File: smartwatch.kicad_pcb (KiCad board)
At the start: 2 copper layers, 40 x 40 mm, 48 parts, among them IC1 LTC4413EDD-1#PBF, IC2 MIA-M10Q-00B, J3 5022441530, J5 Conn_01x04_Socket, U1 NRF52832-QFAA-R, U10 AP2127K-1.8, U2 AP2112K-3.3TRG1, U3 MAX30102, U6 ESP-PSRAM64, U7 MCP73831-2-OT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

Commit message: pcb layout almost complete
Parts:
- removed C10: C, Capacitor_SMD:C_0402_1005Metric
- C9: value C -> 0.8pF
- L1: value L -> 3.9nH; footprint Inductor_SMD:L_0603_1608Metric -> Inductor_SMD:L_0402_1005Metric
- U3, U4, U5: moved to B.Cu
- moved C5 69.0 mm to (189.2, 81.5)
- moved C4 68.0 mm to (187.7, 77.2)
- moved C7 66.4 mm to (186.3, 84.0)
- moved C12 64.1 mm to (187.2, 82.0), turned to 180 degrees
- moved R1 62.8 mm to (180.5, 76.1)
- moved R2 62.8 mm to (180.5, 78.1)
- moved R3 62.8 mm to (180.5, 80.0)
- moved C8 58.7 mm to (183.0, 83.4)
- moved R5 53.0 mm to (171.0, 84.6), turned to -90 degrees
- moved R7 52.3 mm to (169.5, 84.6), turned to -90 degrees
- moved R8 51.4 mm to (166.8, 81.0), turned to 180 degrees
- moved U5 48.4 mm to (168.5, 92.6), turned to 180 degrees
- moved C14 42.2 mm to (164.8, 86.3)
- moved L1 42.0 mm to (166.0, 93.2)
- moved C15 40.1 mm to (167.3, 89.2), turned to 90 degrees
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Connections:
- C9 pad 2: GND -> GNDREF
- U1 pad 15: unconnected-(U1-P0.12-Pad15) -> /SD_CMD
- U1 pad 16: unconnected-(U1-P0.13-Pad16) -> /SRAM_CS
- U1 pad 18: unconnected-(U1-P0.15-Pad18) -> /FLASH_CLK
- U1 pad 19: unconnected-(U1-P0.16-Pad19) -> /SRAM_CMD
- U1 pad 21: unconnected-(U1-P0.18-Pad21) -> /SD_DI
- U1 pad 22: unconnected-(U1-P0.19-Pad22) -> /SRAM_SI02
- U1 pad 23: unconnected-(U1-P0.20-Pad23) -> /SRAM_SIO3
- U1 pad 24: unconnected-(U1-P0.21-Pad24) -> /SRAM_CLK
- U1 pad 31: GND -> GNDREF
- U1 pad 37: unconnected-(U1-P0.25-Pad37) -> /AC_SDA
- U1 pad 38: unconnected-(U1-P0.26-Pad38) -> /AC_SCL
- U1 pad 39: unconnected-(U1-P0.27-Pad39) -> /AC_INT
- U1 pad 4: unconnected-(U1-P0.02-Pad4) -> /GPS_IO
- U1 pad 40: unconnected-(U1-P0.28-Pad40) -> /SRAM_WP
- U1 pad 5: unconnected-(U1-P0.03-Pad5) -> /GPS_RX
- U1 pad 6: unconnected-(U1-P0.04-Pad6) -> /GPS_TX
Routing:
- net Net-(J5-Pin_2): track 0.00 -> 24.6 mm, vias 0 -> 1
- net Net-(J5-Pin_3): track 0.00 -> 23.6 mm, vias 0 -> 1
- net /SWD_VCC: track 0.00 -> 20.7 mm, vias 0 -> 2
- net /AC_SDA: track 0.00 -> 16.2 mm, vias 0 -> 2
- net /AC_INT: track 0.00 -> 16.1 mm
- net /AC_SCL: track 0.00 -> 15.2 mm
- net /SRAM_CS: track 0.00 -> 14.5 mm, vias 0 -> 2
- net /SRAM_CMD: track 0.00 -> 14.2 mm, vias 0 -> 2
- net /SRAM_SI02: track 0.00 -> 13.8 mm, vias 0 -> 2
- net Net-(ANT1-PadFEED): track 0.00 -> 13.5 mm
- net Net-(IC2-RF_IN): track 0.00 -> 9.30 mm
- net /GPS_IO: track 0.00 -> 7.38 mm, vias 0 -> 2
- net /SRAM_CLK: track 0.00 -> 7.23 mm
- net /XC1: track 0.00 -> 7.15 mm
- net /XC2: track 0.00 -> 7.08 mm
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
Commit message: -
Parts:
- removed R8: 3.3k, Resistor_SMD:R_0402_1005Metric
- added C10: 0.8pF, Capacitor_SMD:C_0402_1005Metric, F.Cu at (197.9, 88.0)
- added R4: 800k, Resistor_SMD:R_0402_1005Metric, F.Cu at (195.0, 88.1)
- added R9: 2M, Resistor_SMD:R_0402_1005Metric, F.Cu at (195.0, 90.0)
- U1: footprint NRF52832-QFAA-R:QFN40P600X600X90-49N -> NRF52832-QFAA-R:QFN-48_NOR
- moved R2 19.7 mm to (162.0, 84.7), turned to 90 degrees
- moved U10 13.5 mm to (171.5, 83.5)
- moved C12 12.5 mm to (174.8, 84.0)
- moved C7 11.5 mm to (174.9, 85.1)
- moved C8 8.11 mm to (174.9, 83.0)
- moved R5 5.62 mm to (167.5, 80.2)
- moved R7 5.62 mm to (166.0, 80.2)
- moved U9 4.91 mm to (166.7, 77.3)
- moved C21 1.96 mm to (151.7, 95.1)
- moved J3 0.66 mm to (159.0, 79.3)
- moved C16 0.43 mm to (160.9, 84.7), turned to 90 degrees
- moved U3 0.31 mm to (158.8, 92.6)
Connections:
- R1 pad 1: /HR_SCL -> /AC_SCL
- R3 pad 1: /HR_SDA -> /AC_SDA
- U1 pad 10: unconnected-(U1-P0.08-Pad10) -> /DISPLAY_CS
- U1 pad 11: unconnected-(U1-P0.09-Pad11) -> /DISPLAY_CLK
- U1 pad 12: unconnected-(U1-P0.10-Pad12) -> /DISPLAY_SDI
- U1 pad 14: unconnected-(U1-P0.11-Pad14) -> /FLASH_CS
- U1 pad 17: unconnected-(U1-P0.14-Pad17) -> /TP_SDA
- U1 pad 20: unconnected-(U1-P0.17-Pad20) -> /TP_SCL
- U1 pad 23: /SRAM_SIO3 -> /SD_DO
- U1 pad 24: /SRAM_CLK -> /SD_WP
- U1 pad 27: unconnected-(U1-P0.22-Pad27) -> /SRAM_SIO3
- U1 pad 28: unconnected-(U1-P0.23-Pad28) -> /SRAM_CLK
- U1 pad 29: unconnected-(U1-P0.24-Pad29) -> /SRAM_WP
- U1 pad 39: /AC_INT -> /HR_INT
- U1 pad 40: /SRAM_WP -> unconnected-(U1-P0.28-Pad40)
- U1 pad 42: unconnected-(U1-P0.30-Pad42) -> /TP_RST
- U1 pad 43: unconnected-(U1-P0.31-Pad43) -> /DISPLAY_RESET
- U1 pad 7: unconnected-(U1-P0.05-Pad7) -> /BT_V
- U1 pad 8: unconnected-(U1-P0.06-Pad8) -> /DISPLAY_D/C
- U1 pad 9: unconnected-(U1-P0.07-Pad9) -> /TP_INT
- U3 pad 2: /HR_SCL -> /AC_SCL
- U3 pad 3: /HR_SDA -> /AC_SDA
- U9 pad 12: /AC_INT -> unconnected-(U9-INT1-Pad12)
Routing:
- net /TP_SCL: track 0.00 -> 29.1 mm, vias 0 -> 2
- net /TP_INT: track 0.00 -> 28.9 mm, vias 0 -> 2
- net /TP_SDA: track 0.00 -> 25.6 mm, vias 0 -> 2
- net /DISPLAY_SDI: track 0.00 -> 23.7 mm, vias 0 -> 2
- net /DISPLAY_CLK: track 0.00 -> 22.8 mm, vias 0 -> 2
- net /DISPLAY_D/C: track 0.00 -> 21.8 mm, vias 0 -> 2
- net /DISPLAY_CS: track 0.00 -> 21.2 mm, vias 0 -> 2
- net /AC_INT: track 16.1 -> 0.00 mm
- net /TP_RST: track 0.00 -> 14.1 mm
- net /DISPLAY_RESET: track 0.00 -> 13.6 mm
- net /SD_DO: track 0.00 -> 12.8 mm
- net /SD_WP: track 0.00 -> 12.4 mm
- net /FLASH_CS: track 0.00 -> 11.7 mm
- net /SRAM_WP: track 0.00 -> 8.57 mm
- net Net-(U1-P0.01): track 3.08 -> 10.4 mm
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
Commit message: -
Parts:
- moved U10 1.63 mm to (170.9, 85.0)
- moved C7 0.99 mm to (174.5, 86.0)
- moved C12 0.72 mm to (174.5, 84.7), turned to 0 degrees
- moved C8 0.51 mm to (174.5, 83.3)
Routing:
- net Net-(U10-VOUT): track 0.00 -> 28.9 mm, vias 0 -> 1
- net +3.3V: track 0.00 -> 1.17 mm
Changed lines of the file:
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@@
   )
   (footprint "Package_TO_SOT_SMD:SOT-23-5" (layer "F.Cu")
-    (at 171.5 83.49)
+    (at 170.8875 85)
     (descr "SOT, 5 Pin (https://www.jedec.org/sites/default/files/docs/Mo-178c.PDF variant AA), generated with kicad-footprint-generator ipc_gullwing_generator.py")
     (tags "SOT TO_SOT_SMD")
@@
     (property "ki_keywords" "linear regulator ldo fixed positive")
     (attr smd)
-    (fp_text reference "U10" (at 3.6775 0.066) (layer "F.SilkS")
+    (fp_text reference "U10" (at -3.8 0) (layer "F.SilkS")
         (effects (font (size 1 1) (thickness 0.15)))
     )
@@
   )
   (footprint "Capacitor_SMD:C_0402_1005Metric" (layer "F.Cu")
-    (at 174.8 83.98 180)
+    (at 174.53 84.65)
     (descr "Capacitor SMD 0402 (1005 Metric), square (rectangular) end terminal, IPC_7351 nominal, (Body size source: IPC-SM-782 page 76, https://www.pcb-3d.com/wordpress/wp-content/uploads/ipc-sm-782a_amendment_1_and_2.pdf), generated with kicad-footprint-generator")
     (tags "capacitor")
@@
     (fp_line (start 0.5 0.25) (end -0.5 0.25)
       (stroke (width 0.1) (type solid)) (layer "F.Fab"))
-    (pad "1" smd roundrect (at -0.48 0 180) (size 0.56 0.62) (layers "F.Cu" "F.Paste" "F.Mask") (roundrect_rratio 0.25)
+    (pad "1" smd roundrect (at -0.48 0) (size 0.56 0.62) (layers "F.Cu" "F.Paste" "F.Mask") (roundrect_rratio 0.25)
       (net 14 "Net-(U10-VOUT)") (pintype "passive"))
-    (pad "2" smd roundrect (at 0.48 0 180) (size 0.56 0.62) (layers "F.Cu" "F.Paste" "F.Mask") (roundrect_rratio 0.25)
+    (pad "2" smd roundrect (at 0.48 0) (size 0.56 0.62) (layers "F.Cu" "F.Paste" "F.Mask") (roundrect_rratio 0.25)
       (net 1 "GND") (pintype "passive"))
     (model "${KICAD6_3DMODEL_DIR}/Capacitor_SMD.3dshapes/C_0402_1005Metric.wrl"
@@
   )
   (footprint "Capacitor_SMD:C_0402_1005Metric" (layer "F.Cu")
-    (at 174.87 85.07)
+    (at 174.53 86)
     (descr "Capacitor SMD 0402 (1005 Metric), square (rectangular) end terminal, IPC_7351 nominal, (Body size source: IPC-SM-782 page 76, https://www.pcb-3d.com/wordpress/wp-content/uploads/ipc-sm-782a_amendment_1_and_2.pdf), generated with kicad-footprint-generator")
     (tags "capacitor")
@@
   )
   (footprint "Capacitor_SMD:C_0402_1005Metric" (layer "F.Cu")
-    (at 174.87 82.97)
+    (at 174.53 83.35)
     (descr "Capacitor SMD 0402 (1005 Metric), square (rectangular) end terminal, IPC_7351 nominal, (Body size source: IPC-SM-782 page 76, https://www.pcb-3d.com/wordpress/wp-content/uploads/ipc-sm-782a_amendment_1_and_2.pdf), generated with kicad-footprint-generator")
     (tags "capacitor")
@@
   (via (at 177.5 95.5) (size 0.8) (drill 0.4) (layers "F.Cu" "B.Cu") (free) (net 1))
   (via (at 174 89.75) (size 0.8) (drill 0.4) (layers "F.Cu" "B.Cu") (free) (net 1))
+  (segment (start 157.6 93.42) (end 158.37 93.42) (width 0.3) (layer "B.Cu") (net 2))
+  (segment (start 158.37 93.42) (end 158.65 93.7) (width 0.3) (layer "B.Cu") (net 2))
   (segment (start 154.124314 93.54) (end 154.264314 93.4) (width 0.2) (layer "F.Cu") (net 5))
   (segment (start 154.592053 93.4) (end 154.792053 93.2) (width 0.2) (layer "F.Cu") (net 5))
@@
   (segment (start 154.89 88.625686) (end 157.386 86.129686) (width 0.2) (layer "B.Cu") (net 6))
   (segment (start 157.386 86.129686) (end 157.386 77.744) (width 0.2) (layer "B.Cu") (net 6))
+  (segment (start 173.55 86) (end 174.05 86) (width 0.3) (layer "F.Cu") (net 14))
+  (segment (start 174.05 83.35) (end 173.65 83.35) (width 0.3) (layer "F.Cu") (net 14))
+  (segment (start 173.25 84.95) (end 173.3 85) (width 0.3) (layer "F.Cu") (net 14))
+  (segment (start 173.25 83.75) (end 173.25 84) (width 0.3) (layer "F.Cu") (net 14))
+  (segment (start 173.7 85) (end 174.05 84.65) (width 0.3) (layer "F.Cu") (net 14))
+  (segment (start 173.25 84) (end 173.25 84.95) (width 0.3) (layer "F.Cu") (net 14))
+  (segment (start 173.25 84.95) (end 173.25 85.7) (width 0.3) (layer "F.Cu") (net 14))
+  (segment (start 172.025 84.05) (end 173.2 84.05) (width 0.3) (layer "F.Cu") (net 14))
+  (segment (start 173.2 84.05) (end 173.25 84) (width 0.3) (layer "F.Cu") (net 14))
+  (segment (start 172.4 85) (end 173.3 85) (width 0.3) (layer "F.Cu") (net 14))
+  (segment (start 173.65 83.35) (end 173.25 83.75) (width 0.3) (layer "F.Cu") (net 14))
+  (segment (start 173.3 85) (end 173.7 85) (width 0.3) (layer "F.Cu") (net 14))
+  (segment (start 173.25 85.7) (end 173.55 86) (width 0.3) (layer "F.Cu") (net 14))
+  (via (at 172.4 85) (size 0.8) (drill 0.4) (layers "F.Cu" "B.Cu") (net 14))
+  (segment (start 159.15 95.163718) (end 159.15 92.6) (width 0.3) (layer "B.Cu") (net 14))
+  (segment (start 172.4 85) (end 171.013718 85) (width 0.3) (layer "B.Cu") (net 14))
+  (segment (start 171.013718 85) (end 160.413718 95.6) (width 0.3) (layer "B.Cu") (net 14))
+  (segment (start 159.586282 95.6) (end 159.15 95.163718) (width 0.3) (layer "B.Cu") (net 14))
+  (segment (start 157.62 92.6) (end 157.6 92.62) (width 0.3) (layer "B.Cu") (net 14))
+  (segment (start 159.15 92.6) (end 157.62 92.6) (width 0.3) (layer "B.Cu") (net 14))
+  (segment (start 160.413718 95.6) (end 159.586282 95.6) (width 0.3) (layer "B.Cu") (net 14))
   (segment (start 159.479999 77.841373) (end 159.479999 76.31395) (width 0.2) (layer "F.Cu") (net 15))
   (segment (start 158.8 89.6) (end 158.8 78.521372) (width 0.2) (layer "F.Cu") (net 15))
@@
   (via (at 159.675 97.6) (size 0.5) (drill 0.3) (layers "F.Cu" "B.Cu") (net 19))
   (via (at 162.46 77.49) (size 0.5) (drill 0.3) (layers "F.Cu" "B.Cu") (net 19))
-  (segment (start 159.71 85.46) (end 159.71 80.84) (width 0.2) (layer "B.Cu") (net 19))
-  (segment (start 161.81 78.74) (end 162.3 78.74) (width 0.2) (layer "B.Cu") (net 19))
-  (segment (start 157.79 96.3) (end 157.595686 96.3) (width 0.2) (layer "B.Cu") (net 19))
+  (segment (start 159.64 96.84) (end 159.04 96.84) (width 0.2) (layer "B.Cu") (net 19))
+  (segment (start 160.16 97.36) (end 159.64 96.84) (width 0.2) (layer "B.Cu") (net 19))
+  (segment (start 156.925 89.455) (end 159.71 86.67) (width 0.2) (layer "B.Cu") (net 19))
+  (segment (start 162.82 78.38) (end 162.82 77.85) (width 0.2) (layer "B.Cu") (net 19))
+  (segment (start 156.95 94.62) (end 156.925 94.595) (width 0.2) (layer "B.Cu") (net 19))
   (segment (start 159.675 97.6) (end 160.02 97.6) (width 0.2) (layer "B.Cu") (net 19))
-  (segment (start 159.88 96.84) (end 159.34 96.3) (width 0.2) (layer "B.Cu") (net 19))
-  (segment (start 157.172843 95.877157) (end 156.925 95.629314) (width 0.2) (layer "B.Cu") (net 19))
-  (segment (start 159.71 80.84) (end 161.24 79.31) (width 0.2) (layer "B.Cu") (net 19))
-  (segment (start 160.16 97.46) (end 160.16 97.12) (width 0.2) (layer "B.Cu") (net 19))
-  (segment (start 159.34 96.3) (end 157.79 96.3) (width 0.2) (layer "B.Cu") (net 19))
-  (segment (start 156.925 89.455) (end 157.25 89.13) (width 0.2) (layer "B.Cu") (net 19))
-  (segment (start 157.595686 96.3) (end 157.172843 95.877157) (width 0.2) (layer "B.Cu") (net 19))
+  (segment (start 157.595686 96.3) (end 156.925 95.629314) (width 0.2) (layer "B.Cu") (net 19))
+  (segment (start 161.81 78.74) (end 162.46 78.74) (width 0.2) (layer "B.Cu") (net 19))
+  (segment (start 159.71 80.84) (end 161.81 78.74) (width 0.2) (layer "B.Cu") (net 19))
+  (segment (start 156.925 94.645) (end 156.95 94.62) (width 0.2) (layer "B.Cu") (net 19))
   (segment (start 162.46 78.74) (end 162.82 78.38) (width 0.2) (layer "B.Cu") (net 19))
+  (segment (start 156.925 94.595) (end 156.925 89.455) (width 0.2) (layer "B.Cu") (net 19))
+  (segment (start 160.16 97.46) (end 160.16 97.36) (width 0.2) (layer "B.Cu") (net 19))
+  (segment (start 159.71 86.67) (end 159.71 80.84) (width 0.2) (layer "B.Cu") (net 19))
   (segment (start 162.82 77.85) (end 162.46 77.49) (width 0.2) (layer "B.Cu") (net 19))
-  (segment (start 160.16 97.12) (end 159.88 96.84) (width 0.2) (layer "B.Cu") (net 19))
-  (segment (start 162.3 78.74) (end 162.46 78.74) (width 0.2) (layer "B.Cu") (net 19))
-  (segment (start 156.925 94.645) (end 156.95 94.62) (width 0.2) (layer "B.Cu") (net 19))
-  (segment (start 156.925 94.595) (end 156.925 89.455) (width 0.2) (layer "B.Cu") (net 19))
+  (segment (start 159.04 96.84) (end 158.5 96.3) (width 0.2) (layer "B.Cu") (net 19))
+  (segment (start 156.925 95.629314) (end 156.925 94.645) (width 0.2) (layer "B.Cu") (net 19))
+  (segment (start 158.5 96.3) (end 157.595686 96.3) (width 0.2) (layer "B.Cu") (net 19))
   (segment (start 160.02 97.6) (end 160.16 97.46) (width 0.2) (layer "B.Cu") (net 19))
-  (segment (start 159.71 86.67) (end 159.71 85.46) (width 0.2) (layer "B.Cu") (net 19))
-  (segment (start 156.95 94.62) (end 156.925 94.595) (width 0.2) (layer "B.Cu") (net 19))
-  (segment (start 156.925 95.629314) (end 156.925 94.645) (width 0.2) (layer "B.Cu") (net 19))
-  (segment (start 161.24 79.31) (end 161.81 78.74) (width 0.2) (layer "B.Cu") (net 19))
-  (segment (start 162.82 78.38) (end 162.82 77.85) (width 0.2) (layer "B.Cu") (net 19))
-  (segment (start 157.25 89.13) (end 159.71 86.67) (width 0.2) (layer "B.Cu") (net 19))
   (segment (start 162.45 87.475) (end 162.45 86.11) (width 0.2) (layer "F.Cu") (net 20))
   (segment (start 165.4 78.88) (end 165.9875 78.88) (width 0.2) (layer "F.Cu") (net 20))

Commit message: pcb complete
Parts:
- removed C10: 0.8pF, Capacitor_SMD:C_0402_1005Metric
- removed R5, R7: 3.3k, Resistor_SMD:R_0402_1005Metric
- removed U4, U5: ~, power_pad:power_pad_5mm
- added J1: Conn_01x01_Pin, power_pad:power_pad_5mm, B.Cu at (168.6, 92.6)
- added J2: Conn_01x01_Pin, power_pad:power_pad_5mm, B.Cu at (149.6, 92.6)
- moved R4 29.7 mm to (169.3, 102.9), turned to 180 degrees
- moved R9 27.1 mm to (169.3, 98.8), turned to 180 degrees
- moved C1 25.5 mm to (145.7, 105.4), turned to 180 degrees
- moved C5 17.7 mm to (171.5, 80.5)
- moved C4 16.3 mm to (171.6, 79.2)
- moved R1 15.1 mm to (166.0, 80.3), turned to -90 degrees
- moved R3 13.0 mm to (167.5, 80.3), turned to -90 degrees
- moved C21 2.65 mm to (149.1, 94.7)
- moved C15 1.79 mm to (169.1, 89.0)
- moved X1 1.79 mm to (166.8, 88.5)
- moved C14 1.77 mm to (166.5, 86.2)
- moved BT1 1.17 mm to (172.9, 100.9)
- moved R6 0.69 mm to (143.0, 101.2)
- moved C2 0.64 mm to (147.1, 99.4), turned to 180 degrees
- moved C11 0.49 mm to (154.8, 88.7)
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Connections:
- C16 pad 1: Power Supply -> +3.3V
- C20 pad 1: Power Supply -> +3.3V
- C21 pad 1: Power Supply -> +3.3V
- C6 pad 1: Power Supply -> +3.3V
- C9 pad 2: GNDREF -> GND
- U1 pad 13: Power Supply -> +3.3V
- U1 pad 31: GNDREF -> GND
- U1 pad 32: GND -> unconnected-(U1-DEC2-Pad32)
- U1 pad 36: Power Supply -> +3.3V
- U1 pad 48: Power Supply -> +3.3V
- U2 pad 5: Power Supply -> +3.3V
Routing:
- net +3.3V: track 1.17 -> 197.0 mm, vias 0 -> 18
- net Net-(BT1-+): track 0.00 -> 43.1 mm, vias 0 -> 4
- net /BT_V: track 1.88 -> 38.7 mm, vias 1 -> 4
- net Net-(U1-P0.00): track 9.77 -> 29.3 mm, vias 0 -> 4
- net /AC_SDA: track 15.3 -> 30.7 mm, vias 2 -> 1
- net Power Supply: track 10.9 -> 0.00 mm, vias 2 -> 0
- net /AC_SCL: track 14.9 -> 24.9 mm, vias 0 -> 1
- net /SWD_VCC: track 20.7 -> 30.6 mm, vias 2 -> 3
- net GND: track 4.06 -> 11.7 mm, vias 26 -> 75
- net /HR_INT: track 5.08 -> 10.8 mm, vias 0 -> 1
- net /DISPLAY_CS: track 21.2 -> 26.9 mm
- net Net-(U1-P0.01): track 10.4 -> 15.3 mm, vias 0 -> 2
- net unconnected-(U1-P0.29-Pad41): track 3.01 -> 0.00 mm
- net unconnected-(U1-P0.28-Pad40): track 2.99 -> 0.00 mm
- net GNDREF: track 2.31 -> 0.00 mm
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Other:
- board text added: "BL"
- board text added: "DS"
- board text added: "Designed By - Iiro Karppanen -"
- board text added: "GPS"
- board text added: "SWD"
