File: smartwatch.kicad_sch (KiCad schematic)
At the start: 47 parts, among them IC2 NORA-B120-00B, J1 Power_Pad-, J2 Power_Pad+, J3 5022441530, J5 Conn_01x06_Pin, Q1 2N7002-7-F, Q2 Q_PMOS_DGS, U1 MAX17048G+T10, U10 AP2127K-1.8, U2 AP2112K-3.3TRG1, U3 MAX30102, U4 DS1302Z+T&R, U5 CAM-M8C-0, U7 MCP73831-2-OT, U8 W25Q128JVS, U9 LIS2DE12, X2 9HT10-32.768KBZC-T, Y1 32.768kHz

Commit message: charging circuit complete
Parts:
- removed BT1: Battery_Cell, Capacitor_SMD:C_1812_4532Metric, symbol Device:Battery_Cell
- removed C10, C6: 100uF, Capacitor_SMD:C_0402_1005Metric, symbol Device:C
- removed C11: 0.1uF, Capacitor_SMD:C_0402_1005Metric, symbol Device:C
- removed C2: 1uF, Capacitor_SMD:C_0402_1005Metric, symbol Device:C
- removed D1: LED_GREEN, LED_SMD:LED_0402_1005Metric, symbol Device:LED
- removed D4: D_Schottky, symbol Device:D_Schottky
- removed J5: Conn_01x06_Pin, Connector_PinHeader_2.54mm:PinHeader_1x06_P2.54mm_Vertical, symbol Connector:Conn_01x06_Pin
- removed Q2: Q_PMOS_DGS, symbol Device:Q_PMOS_DGS
- removed R1: 10k, symbol Device:R
- removed R12: 470, Resistor_SMD:R_0402_1005Metric, symbol Device:R
- removed R4, R9: 3.3k, Resistor_SMD:R_0603_1608Metric, symbol Device:R
- removed R6: 5.1k, Resistor_SMD:R_0402_1005Metric, symbol Device:R
- removed U2: AP2112K-3.3TRG1, AP2112K-3-3TRG1:SOT_RG1_DIO, symbol AP2112K-3-3TRG1:AP2112K-3.3TRG1
- removed U7: MCP73831-2-OT, Package_TO_SOT_SMD:SOT-23-5, symbol Battery_Management:MCP73831-2-OT
- removed U8: W25Q128JVS, Package_SO:SOIC-8_5.23x5.23mm_P1.27mm, symbol Memory_Flash:W25Q128JVS
- added BT3: Battery_Cell, Capacitor_SMD:C_1812_4532Metric, symbol Device:Battery_Cell
- added C15: 100uF, Capacitor_SMD:C_0402_1005Metric, symbol Device:C
- added C16: 4.7uF, Capacitor_Tantalum_SMD:CP_EIA-2012-12_Kemet-R, symbol Device:C
- added C18: 0.1uF, Capacitor_SMD:C_0402_1005Metric, symbol Device:C
- added C19: 4.7uF, Capacitor_SMD:C_0402_1005Metric, symbol Device:C
- added D6: LED_GREEN, LED_SMD:LED_0402_1005Metric, symbol Device:LED
- added IC1: W25N01GVZEIG, SON127P800X600X80-9N-D, symbol W25N01GVZEIG_TR:W25N01GVZEIG_TR
- added J4: Conn_01x03_Pin, Connector_PinSocket_2.54mm:PinSocket_1x03_P2.54mm_Vertical, symbol Connector:Conn_01x03_Pin
- added J6: Conn_01x01_Pin, Connector_PinSocket_2.54mm:PinSocket_1x01_P2.54mm_Vertical, symbol Connector:Conn_01x01_Pin
- added Q2, Q6: NTR1P02T1G, Package_TO_SOT_SMD:SOT-23, symbol Device:Q_PMOS_DSG
- added R13, R14: 3.3k, Resistor_SMD:R_0603_1608Metric, symbol Device:R
- added R16: 5.1k, Resistor_SMD:R_0603_1608Metric, symbol Device:R
- added R17: 5.1k, Resistor_SMD:R_0402_1005Metric, symbol Device:R
- added R18: 470, Resistor_SMD:R_0402_1005Metric, symbol Device:R
- added U11: MCP73831-2-OT, Package_TO_SOT_SMD:SOT-23-5, symbol Battery_Management:MCP73831-2-OT
- added U8: AP2112K-3.3TRG1, AP2112K-3-3TRG1:SOT_RG1_DIO, symbol AP2112K-3-3TRG1:AP2112K-3.3TRG1
- C1: value 4.7uF -> 1uF
- D5: value D_Schottky -> LBAT54XV2T1G; footprint (none) -> Diode_SMD:D_SOD-523
- J1: value Power_Pad- -> Charging_Pad-
- J2: value Power_Pad+ -> Charging_Pad+
- Q1: value 2N7002-7-F -> 2N7002
Connections:
- net BACKLIGHT_EN: now also IC2.E8 (P0.05/AIN1_)
- net FLASH_CLK: now also IC2.F1 (P0.17/SCK), IC1.6 (CLK)
- net FLASH_CS: now also IC2.E1 (P0.18/CSN), IC1.1 (~{CS})
- net GND: now also BT3.2 (-), C15.2, C16.2, C18.2, C19.2, IC1.4 (GND), IC1.9 (EP), R16.2, R17.1, U11.2 (V_{SS}), U8.2 (GND)
- net RESET_N: now also J6.1 (Pin_1)
- net SCL: now also IC2.G9 (P1.13), R14.1
- net SDA: now also IC2.H9 (P1.11_), R13.1
- net SWDCLK: now also J4.2 (Pin_2)
- net SWDIO: now also J4.1 (Pin_1)
- net SWO: now also J4.3 (Pin_3)
- net VBUS: now also C1.1, D5.2 (A), J2.1 (Pin_1), Q2.3 (G), Q6.3 (G), R16.1, R18.1, U11.4 (V_{DD})
- net VSYS: now also C15.1, C16.1, IC1.8 (VCC), R13.2, R14.2, U8.5 (VOUT); no longer U10.1 (VIN)
- net at D5.1 (K): now also Q2.2 (S), U8.1 (VIN), U8.3 (EN)
- net BAT+: now reaches U1.2 (CELL), U1.3 (VDD)
- net BAT+: now also U10.1 (VIN), BT3.1 (+), C18.1, C19.1, Q6.2 (S), U11.3 (V_{BAT}); no longer C1.1
- net FLASH_IO2: now reaches IC2.D1 (P0.15/IO2)
- net FLASH_IO2: now also IC1.3 (~{WP_(IO2)})
- net FLASH_IO0: now reaches IC2.D2 (P0.13/IO0)
- net FLASH_IO0: now also IC1.5 (DI_(IO0))
- net FLASH_IO1: now reaches IC2.E2 (P0.14/IO1)
- net FLASH_IO1: now also IC1.2 (DO_(IO1))
- net FLASH_IO3: now reaches IC2.F2 (P0.16/IO3)
- net FLASH_IO3: now also IC1.7 (~{HOLD_(IO3)})
- new net: R17.2, U11.5 (PROG)
- new net: D6.1 (K), U11.1 (STAT)
- new net: Q2.1 (D), Q6.1 (D)
- new net: D6.2 (A), R18.2
Other:
- note added: "Battery Gauge"
- note added: "Display"
- note added: "Power"
- note removed: "Charging and Power Delivery Circuit"
- note removed: "Display Connector"
- moved on the sheet: J1, J2, U1, U4, U9, Y1
