File: Hardware/smartwatch.kicad_pcb (KiCad board)
At the start: 4 copper layers, 38 x 38 mm, 54 parts, among them IC1 W25N01GVZEIG, IC2 NORA-B120-00B, IC3 LM66200DRLR, J1 Charging_Pad-, J2 Charging_Pad+, J3 DS1020-09-15VBT1A, J4 Conn_01x04_Pin, Q1 2N7002, U1 MAX17048G+T10, U11 MCP73831T-2ACI/OT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

Commit message: -
Parts:
- removed J1: Charging_Pad-, power_pad:power_pad_4mm
- removed J2: Charging_Pad+, power_pad:power_pad_4mm
- removed Q1: 2N7002, Package_TO_SOT_SMD:SOT-23-3
- removed R16, R20: 4.7k, Resistor_SMD:R_0402_1005Metric
- removed REF** (x2): MountingHole_2.2mm_M2, MountingHole:MountingHole_2.2mm_M2
- added J5: MEM2075-00-140-01-A, MEM2075_00_140_01_A:GCT_MEM2075-00-140-01-A, B.Cu at (155.4, 101.2)
- added MOSFET1: 2N7002, 2N7002:SOT-23TO-236_318-08_ONS, F.Cu at (139.5, 85.1)
- added U7: BMI270, BMI270:BMI270_BOS, F.Cu at (93.7, 121.6)
- added U8: LIS2MDLTR, LIS2MDLTR:LGA-12_2X2X1_STM, F.Cu at (93.1, 125.4)
- IC1: value W25N01GVZEIG -> W25Q256JVEIQ
- J3: value DS1020-09-15VBT1A -> DF37NB-24DS-0.4V51; footprint DISPLAY_CONNECTOR:FPC-SMD_P0.50-15P_LSXJ-H2.0-15P -> DF37NB_24DS_0_4V_51_:CONN_DF37NB-24DS-0.4V51_HIR
- moved U9 83.7 mm to (97.7, 133.5)
- moved X2 81.0 mm to (93.4, 133.4), turned to 0 degrees
- moved R13 68.5 mm to (117.7, 131.7)
- moved R19 67.5 mm to (109.6, 118.7), turned to 0 degrees
- moved R14 65.8 mm to (117.7, 134.2), turned to 0 degrees
- moved C5 64.3 mm to (103.8, 132.6), turned to 0 degrees
- moved R6 64.2 mm to (103.8, 120.7), turned to 0 degrees
- moved R12 62.8 mm to (106.7, 120.7), turned to 0 degrees
- moved R15 62.8 mm to (106.7, 122.7), turned to 0 degrees
- moved C4 62.3 mm to (103.8, 130.6), turned to 0 degrees
- moved C18 62.1 mm to (109.5, 130.6), turned to 0 degrees
- moved R2 60.2 mm to (117.7, 124.2)
- moved U2 60.2 mm to (122.2, 125.3), turned to 0 degrees
- moved R4 59.9 mm to (103.8, 116.7), turned to 0 degrees
- moved R21 56.0 mm to (109.6, 120.7), turned to 0 degrees
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Connections:
- IC1 pad 1: /FLASH_CS -> unconnected-(IC1-~{CS}-Pad1)
- IC1 pad 2: /FLASH_IO1 -> unconnected-(IC1-DO_(IO1)-Pad2)
- IC1 pad 3: /FLASH_IO2 -> unconnected-(IC1-~{WP_(IO2)}-Pad3)
- IC1 pad 4: GND -> unconnected-(IC1-GND-Pad4)
- IC1 pad 5: /FLASH_IO0 -> unconnected-(IC1-DI_(IO0)-Pad5)
- IC1 pad 6: /FLASH_CLK -> unconnected-(IC1-CLK-Pad6)
- IC1 pad 7: /FLASH_IO3 -> unconnected-(IC1-~{HOLD_(IO3)}-Pad7)
- IC1 pad 8: +3.3V -> unconnected-(IC1-VCC-Pad8)
- IC1 pad 9: GND -> unconnected-(IC1-EP-Pad9)
- J3 pad 1: GND -> /LEDK
- J3 pad 10: GND -> /DISPLAY_RESET
- J3 pad 11: GND -> +3.3V
- J3 pad 12: /TP_RST -> +3.3V
- J3 pad 13: /TP_INT -> +3.3V
- J3 pad 14: /TP_SDA -> +3.3V
- J3 pad 15: /TP_SCL -> GND
- J3 pad 16: (no net) -> GND
- J3 pad 17: (no net) -> +3.3V
- J3 pad 3: Net-(J3-Pad3) -> GND
- J3 pad 4: +3.3V -> GND
- J3 pad 6: /DISPLAY_CS -> /DISPLAY_SDI
- J3 pad 7: /DISPLAY_CLK -> /DISPLAY_SD0
- J3 pad 8: /DISPLAY_SDI -> /DISPLAY_CLK
- J3 pad 9: /DISPLAY_RESET -> /DISPLAY_CS
- R19 pad 2: /BAT+ -> +3.3V
- R2 pad 2: Net-(J3-Pad3) -> unconnected-(R2-Pad2)
- R21 pad 1: /FLASH_IO3 -> unconnected-(R21-Pad1)
- R21 pad 2: +3.3V -> unconnected-(R21-Pad2)
- U2 pad 6: /BAT+ -> +3.3V
- U2 pad 7: /BAT+ -> +3.3V
Routing:
- net +3.3V: track 143.2 -> 88.5 mm, vias 13 -> 1
- net /SCL: track 51.8 -> 0.00 mm, vias 5 -> 0
- net /SDA: track 48.8 -> 0.00 mm, vias 5 -> 0
- net /BAT+: track 76.0 -> 35.3 mm, vias 4 -> 0
- net /BACKLIGHT_EN: track 29.1 -> 0.00 mm, vias 2 -> 0
- net /SWDIO: track 24.0 -> 0.00 mm, vias 1 -> 0
- net /RESET_N: track 23.3 -> 0.00 mm, vias 1 -> 0
- net +1V8: track 29.9 -> 6.61 mm, vias 2 -> 0
- net /SWDCLK: track 22.4 -> 0.00 mm, vias 1 -> 0
- net /TP_SDA: track 22.3 -> 0.00 mm, vias 2 -> 0
- net /TP_SCL: track 22.1 -> 0.00 mm, vias 2 -> 0
- net /TP_INT: track 21.0 -> 0.00 mm, vias 2 -> 0
- net /TP_RST: track 20.7 -> 0.00 mm, vias 2 -> 0
- net /RTC_INT: track 18.9 -> 0.00 mm, vias 3 -> 0
- net /GPS_EXTINT: track 18.7 -> 0.00 mm
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Other:
- board text removed: "+"
- board text removed: "-"
- board text removed: "Designed by Iiro Karppanen"
