File: Hardware/smartwatch.kicad_pcb (KiCad board)
At the start: 4 copper layers, 35 x 38.6 mm, 56 parts, among them IC1 W25Q256JVEIQ, IC2 NORA-B120-00B, IC3 LM66200DRLR, J1 Conn_01x04, J2 Conn_01x04, J3 DF37NB-24DS-0.4V51, U1 MAX17048G+T10, U11 MCP73831T-2ACI/OT, U2 TPD2EUSB30DRTR, U3 MAX30102, U4 TPS63031DSK, U5 L96-M33, U6 AP7313-18SAG-7, U7 BMI270, U8 LIS2MDLTR, U9 TPD2EUSB30DRTR, X2 9HT10-32.768KBZC-T

Commit message: final version
Parts:
- removed BT4: 2994TR, 2994TR:BAT_2994TR
- removed D1: LED_GREEN, LED_SMD:LED_0402_1005Metric
- removed J3: DF37NB-24DS-0.4V51, DF37NB_24DS_0_4V_51_:CONN_DF37NB-24DS-0.4V51_HIR
- removed R18: 470, Resistor_SMD:R_0402_1005Metric
- removed REF** (x2): MountingHole_2.2mm_M2, MountingHole:MountingHole_2.2mm_M2
- added BT2: 2994TR, 2994TR:BAT_2994TR, F.Cu at (151.5, 113.3)
- added C17: 100nF, Capacitor_SMD:C_0402_1005Metric, F.Cu at (148.1, 89.5)
- added C20: 4.7uF, Capacitor_SMD:C_0402_1005Metric, F.Cu at (148.1, 90.5)
- added C21: 2.2uF, Capacitor_SMD:C_0402_1005Metric, F.Cu at (162.8, 115.9)
- added C22: 1uF, Capacitor_SMD:C_0402_1005Metric, F.Cu at (165.7, 115.2)
- added C23: 1uF, Capacitor_SMD:C_0402_1005Metric, F.Cu at (171.1, 111.8)
- added IC4: LM66200DRLR, LM66200DRLR:SOTFL50P160X60-8N, F.Cu at (154.7, 109.6)
- added J4: X05A20L15T, X05A20L15T:CONN_X05A20L15T_XKB, F.Cu at (159.2, 85.1)
- added R10: 4.7k, Resistor_SMD:R_0402_1005Metric, F.Cu at (167.8, 86.7)
- added R12: 4.7k, Resistor_SMD:R_0402_1005Metric, F.Cu at (156.3, 80.6)
- added R15: 4.7k, Resistor_SMD:R_0402_1005Metric, F.Cu at (165.5, 89.2)
- added R16: 4.7k, Resistor_SMD:R_0402_1005Metric, F.Cu at (154.5, 81.1)
- added U10: RV-3028-C7_32.768KHZ_1PPM-TA-QC, RV_3028_C7_32_768KHZ_1PPM_TA_QC:IC_RV-3028-C7_32.768KHZ_1PPM-TA-QC, F.Cu at (173.7, 90.8)
- added U12: TPS70950QDRVRQ1, TPS70950QDRVRQ1:DRV0006A, F.Cu at (164.1, 113.0)
- BT1: footprint 78171-0002:78171-0002 -> Capacitor_SMD:C_1812_4532Metric_Pad1.57x3.40mm_HandSolder
- C16: value 4.7uF -> 1uF
- C7: value 0.1uF -> 4.7uF
- C8: value 4.7uF -> 0.1uF
- J1: footprint Pogo_Female_4pin:Pogo_Female_4Pin -> Pogo_Female_4Pin:Pogo_Female_4Pin
- R13: value 4.7k -> 1k
- R14: value 4.7k -> 5k6
- U3: value MAX30102 -> MAX30101EFD_T; footprint OptoDevice:Maxim_OLGA-14_3.3x5.6mm_P0.8mm -> MAX30101EFD_T:MAX30101EFD_T
- moved C14 46.2 mm to (144.3, 88.6), turned to 180 degrees
- moved C13 43.9 mm to (146.6, 90.0), turned to -90 degrees
- moved C7 36.1 mm to (161.3, 90.4), turned to 90 degrees
- moved C8 35.3 mm to (160.3, 90.4), turned to 90 degrees
- moved C4 32.9 mm to (159.2, 101.0)
- moved C5 32.2 mm to (159.2, 99.9)
- moved R9 27.1 mm to (157.3, 90.2), turned to 90 degrees
- moved C16 25.0 mm to (162.7, 109.9), turned to 0 degrees
- moved U7 21.1 mm to (147.7, 86.4), turned to 0 degrees
- moved J1 20.2 mm to (163.3, 88.2), turned to 180 degrees
- moved C11 16.0 mm to (169.0, 88.2), turned to -90 degrees
- moved J2 15.6 mm to (155.2, 108.4), turned to 0 degrees
- moved C12 14.6 mm to (170.7, 90.3), turned to -135 degrees
- moved U1 13.9 mm to (151.4, 86.5), turned to 90 degrees
- moved C3 13.7 mm to (170.1, 88.2), turned to -90 degrees
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Connections:
- C16 pad 1: +3.3V -> VDD
- C4 pad 1: +3.3V -> +5V
- C5 pad 1: +3.3V -> +5V
- C9 pad 1: VBUS -> VDD
- IC2 pad A2: /GPS_EXTINT -> unconnected-(IC2-P0.12/TRACECLK/DCX-PadA2)
- IC2 pad A3: unconnected-(IC2-P1.03/TWI-PadA3) -> /TWI_SCL
- IC2 pad A4: /GPS_TX -> /GPS_RX
- IC2 pad A5: /GPS_RX -> /GPS_TX
- IC2 pad B4: unconnected-(IC2-P1.02/TWI-PadB4) -> /TWI_SDA
- IC2 pad B5: /GPS_EXTINT -> unconnected-(IC2-P0.03/NFC2-PadB5)
- IC2 pad B9: VIN_SWD -> VIN_USB
- IC2 pad C4: unconnected-(IC2-P1.01-PadC4) -> /GPS_EXTINT
- IC2 pad C5: unconnected-(IC2-P0.02/NFC1-PadC5) -> /GPS_FORCEON
- IC2 pad D7: /TP_SCL -> /HR_INT
- IC2 pad D8: /TP_INT -> unconnected-(IC2-P0.04/AIN0-PadD8)
- IC2 pad E7: /TP_SDA -> /DISPLAY_CS
- IC2 pad E9: unconnected-(IC2-P1.05-PadE9) -> /TP_INT
- IC2 pad F3: unconnected-(IC2-P0.19-PadF3) -> /HR_LED_EN
- IC2 pad F4: unconnected-(IC2-VSS_7-PadF4) -> GND
- IC2 pad F5: unconnected-(IC2-VSS_8-PadF5) -> GND
- IC2 pad F7: /DISPLAY_RESET -> /DISPLAY_CLK
- IC2 pad F9: unconnected-(IC2-P1.15-PadF9) -> /DISPLAY_RESET
- IC2 pad G3: unconnected-(IC2-P0.25/AIN4-PadG3) -> /INT1_BMI270
- IC2 pad G4: /BAT_INT -> /INT2_BMI270
- IC2 pad G8: /DISPLAY_CLK -> unconnected-(IC2-P1.12-PadG8)
- IC2 pad H3: unconnected-(IC2-P0.27/AIN6-PadH3) -> /LIS2MDLTR_INT
- IC2 pad H7: /DISPLAY_CS -> /BAT_INT
- IC2 pad J3: /LIS2MDLTR_INT -> unconnected-(IC2-RESET_N-PadJ3)
- IC2 pad J4: /INT1_BMI270 -> unconnected-(IC2-N/C_3-PadJ4)
- IC2 pad J5: /INT2_BMI270 -> unconnected-(IC2-N/C_4-PadJ5)
- IC3 pad 2: VBUS -> VDD
- IC3 pad 3: VIN_SWD -> VIN
- IC3 pad 7: VBUS -> VDD
- J1 pad 1: VIN_SWD -> VIN_USB
- R13 pad 1: /SDA -> /GPS_FORCEON
- R13 pad 2: +1V8 -> Net-(U5-FORCE_ON)
- R14 pad 1: /SCL -> Net-(U5-FORCE_ON)
- R14 pad 2: +1V8 -> GND
- R2 pad 1: Net-(U5-RF_OUT) -> Net-(U5-RF_IN)
- R2 pad 2: Net-(U5-RF_IN) -> Net-(U5-RF_OUT)
- R9 pad 2: +3.3V -> +1V8
- U11 pad 1: Net-(U11-STAT) -> GND
- U11 pad 4: VIN_SWD -> VIN
- U3 pad 1: unconnected-(U3-NC-Pad1) -> (no net)
- U3 pad 10: +3.3V -> +5V
- U3 pad 14: unconnected-(U3-NC-Pad14) -> (no net)
- U3 pad 2: /SCL -> /TWI_SCL
- U3 pad 3: /SDA -> /TWI_SDA
- U3 pad 5: unconnected-(U3-NC-Pad5) -> (no net)
- U3 pad 6: unconnected-(U3-NC-Pad6) -> (no net)
- U3 pad 7: unconnected-(U3-NC-Pad7) -> (no net)
- U3 pad 8: unconnected-(U3-NC-Pad8) -> (no net)
- U3 pad 9: +3.3V -> +5V
- U4 pad 5: VBUS -> VDD
- U5 pad 28: unconnected-(U5-FORCE_ON-Pad28) -> Net-(U5-FORCE_ON)
- U6 pad 1: VBUS -> VDD
Routing:
- net +1V8: track 0.64 -> 99.8 mm, vias 1 -> 8
- net RTC Battery: track 0.00 -> 87.8 mm, vias 0 -> 3
- net +3.3V: track 51.2 -> 113.1 mm, vias 4 -> 9
- net /TWI_SDA: track 0.00 -> 47.3 mm, vias 0 -> 2
- net /INT1_BMI270: track 2.41 -> 49.3 mm, vias 1 -> 2
- net +5V: track 0.00 -> 44.2 mm, vias 0 -> 2
- net /INT2_BMI270: track 2.25 -> 46.0 mm, vias 1 -> 2
- net /TWI_SCL: track 0.00 -> 42.4 mm, vias 0 -> 2
- net /BAT_INT: track 0.00 -> 38.1 mm, vias 0 -> 2
- net /SCL: track 17.7 -> 50.7 mm, vias 0 -> 5
- net VIN_USB: track 0.00 -> 31.4 mm, vias 0 -> 3
- net GND: track 0.00 -> 30.1 mm, vias 21 -> 78
- net /BAT+: track 18.5 -> 48.5 mm, vias 2 -> 3
- net /SWDIO: track 0.00 -> 26.4 mm, vias 0 -> 1
- net /HR_LED_EN: track 0.00 -> 26.2 mm, vias 0 -> 2
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Other:
- board size 35 x 38.6 mm -> 35 x 38.5 mm

Commit message: -
Parts:
- added REF**: Nordic_AQFN-73-1EP_7x7mm_P0.5mm, Package_DFN_QFN:Nordic_AQFN-73-1EP_7x7mm_P0.5mm, F.Cu at (233.2, 95.4)
Other:
- board size 35 x 38.5 mm -> 98.7 x 42 mm

Commit message: -
Parts:
- removed REF**: Nordic_AQFN-73-1EP_7x7mm_P0.5mm, Package_DFN_QFN:Nordic_AQFN-73-1EP_7x7mm_P0.5mm
- added E1: W3010, W3010:XCVR_W3010, F.Cu at (221.7, 106.8)
- added U13: MIA-M10Q-00B, MIA-M10Q-00B:LGA_M10Q-00B_UBL, F.Cu at (230.2, 108.2)
- C11, C12, C13, C14, C18, C3: footprint Capacitor_SMD:C_0402_1005Metric -> Capacitor_SMD:C_0201_0603Metric
- J1, U3: moved to F.Cu
- J2: footprint Pogo_Female_4pin:Pogo_Female_4Pin -> Pogo_Female_4Pin:Pogo_Female_4Pin; moved to F.Cu
- R10, R12, R15, R16: footprint Resistor_SMD:R_0402_1005Metric -> Resistor_SMD:R_0201_0603Metric
- moved U11 99.5 mm to (243.9, 130.8)
- moved R16 97.3 mm to (245.1, 116.8)
- moved R12 95.3 mm to (245.1, 115.1), turned to 0 degrees
- moved U7 94.5 mm to (239.3, 109.7), turned to -90 degrees
- moved C14 91.3 mm to (233.9, 105.9)
- moved BT2 89.9 mm to (238.0, 137.8), turned to 35 degrees
- moved L2 89.6 mm to (243.1, 134.3), turned to 90 degrees
- moved C13 88.9 mm to (233.9, 106.7), turned to 180 degrees
- moved J4 87.5 mm to (227.2, 140.3), turned to 180 degrees
- moved U1 86.4 mm to (234.5, 110.0), turned to 180 degrees
- moved IC3 85.3 mm to (239.9, 131.0), turned to 0 degrees
- moved R15 83.9 mm to (245.1, 115.9), turned to 0 degrees
- moved C18 83.7 mm to (233.9, 107.5)
- moved R10 82.0 mm to (245.1, 114.3), turned to 0 degrees
- moved BT1 81.3 mm to (232.7, 148.1), turned to 180 degrees
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Connections:
- R8 pad 1: GND -> Net-(U5-EXTINT0)
- R8 pad 2: Net-(U5-EXTINT0) -> GND
Routing:
- net +3.3V: track 113.1 -> 0.00 mm, vias 9 -> 0
- net +1V8: track 99.8 -> 0.00 mm, vias 8 -> 0
- net RTC Battery: track 87.8 -> 0.00 mm, vias 3 -> 0
- net /SCL: track 50.7 -> 0.00 mm, vias 5 -> 0
- net /INT1_BMI270: track 49.3 -> 0.00 mm, vias 2 -> 0
- net /BAT+: track 48.5 -> 0.00 mm, vias 3 -> 0
- net /TWI_SDA: track 47.3 -> 0.00 mm, vias 2 -> 0
- net /INT2_BMI270: track 46.0 -> 0.00 mm, vias 2 -> 0
- net +5V: track 44.2 -> 0.00 mm, vias 2 -> 0
- net /SDA: track 43.0 -> 0.00 mm, vias 2 -> 0
- net /TWI_SCL: track 42.4 -> 0.00 mm, vias 2 -> 0
- net /BAT_INT: track 38.1 -> 0.00 mm, vias 2 -> 0
- net VIN_USB: track 31.4 -> 0.00 mm, vias 3 -> 0
- net GND: track 30.1 -> 0.89 mm, vias 78 -> 1
- net /SWDIO: track 26.4 -> 0.00 mm, vias 1 -> 0
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Other:
- board size 98.7 x 42 mm -> 38.2 x 41.9 mm
