File: Hardware/smartwatch.kicad_sch (KiCad schematic)
At the start: 56 parts, among them IC1 W25Q256JVEIQ, IC2 NORA-B120-00B, IC3 LM66200DRLR, J1 Conn_01x04, J2 Conn_01x04, J3 DF37NB-24DS-0.4V51, J4 5022441530, U1 MAX17048G+T10, U10 RV-3028-C7_32.768KHZ_1PPM-TA-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, U11 MCP73831T-2ACI/OT, U2 TPD2EUSB30DRTR, U3 MAX30102, U4 TPS63031DSK, U5 L96-M33, U6 AP7313-18SAG-7, U7 BMI270, U8 LIS2MDLTR, U9 TPD2EUSB30DRTR, X2 9HT10-32.768KBZC-T

Commit message: final version
Parts:
- removed D1: LED_GREEN, LED_SMD:LED_0402_1005Metric, symbol Device:LED
- removed J3: DF37NB-24DS-0.4V51, CONN_DF37NB-24DS-0.4V51_HIR, symbol DF37NB_24DS_0_4V_51_:DF37NB-24DS-0.4V51
- removed J4: 5022441530, CONN_502244-1530_MOL, symbol MOLEX_5022441530:5022441530
- removed R18: 470, Resistor_SMD:R_0402_1005Metric, symbol Device:R
- removed U3: MAX30102, OptoDevice:Maxim_OLGA-14_3.3x5.6mm_P0.8mm, symbol Sensor:MAX30102
- added C17: 100nF, Capacitor_SMD:C_0402_1005Metric, symbol Device:C
- added C20: 4.7uF, Capacitor_SMD:C_0402_1005Metric, symbol Device:C
- added C21: 2.2uF, Capacitor_SMD:C_0402_1005Metric, symbol Device:C
- added C22, C23: 1uF, Capacitor_SMD:C_0402_1005Metric, symbol Device:C
- added IC4: LM66200DRLR, LM66200DRLR:SOTFL50P160X60-8N, symbol LM66200DRLR:LM66200DRLR
- added J4: X05A20L15T, X05A20L15T:CONN_X05A20L15T_XKB, symbol X05A20L15T:X05A20L15T
- added R10, R12, R15, R16: 4.7k, Resistor_SMD:R_0402_1005Metric, symbol Device:R
- added U12: TPS70950QDRVRQ1, DRV0006A, symbol TPS70950QDRVRQ1:TPS70950QDRVRQ1
- added U3: MAX30101EFD_T, MAX30101EFD_T:MAX30101EFD_T, symbol MAX30101EFD_T:MAX30101EFD_T
- BT1: footprint 78171-0002:78171-0002 -> Capacitor_SMD:C_1812_4532Metric_Pad1.57x3.40mm_HandSolder
- C16: value 4.7uF -> 1uF
- C7: value 0.1uF -> 4.7uF
- C8: value 4.7uF -> 0.1uF
- J1, J2: footprint Pogo_Female_4pin:Pogo_Female_4Pin -> Pogo_Female_4Pin:Pogo_Female_4Pin
- R13: value 4.7k -> 1k; MPN NRF52840-QIAA-R -> (none)
- R14: value 4.7k -> 5k6; MPN NRF52840-QIAA-R -> (none)
- U10: footprint RV-3028-C7_32.768KHZ_1PPM-TA-QC:IC_RV-3028-C7_32.768KHZ_1PPM-TA-QC -> RV_3028_C7_32_768KHZ_1PPM_TA_QC:IC_RV-3028-C7_32.768KHZ_1PPM-TA-QC
Connections:
- net TP_SCL is gone; now on net HR_INT: IC2.D7 (P0.23)
- net TP_SDA is gone; now on net DISPLAY_CS: IC2.E7 (P0.06/AIN2)
- net +1V8: now also R9.2, C23.1, R10.2, R15.2, U3.11 (VDD); no longer R13.2, R14.2
- net +3.3V: now also J4.12, J4.13, J4.6, R12.1, R16.1; no longer C16.1, C4.1, C5.1, R9.2
- net BAT_INT: now also IC2.H7 (P0.29); no longer IC2.G4 (P1.04)
- net DISPLAY_CLK: now also IC2.F7 (P1.07), J4.9; no longer IC2.G8 (P1.12)
- net DISPLAY_CS: now also J4.10; no longer IC2.H7 (P0.29)
- net DISPLAY_D/C: now also J4.11
- net DISPLAY_RESET: now also IC2.F9 (P1.15), J4.7; no longer IC2.F7 (P1.07)
- net DISPLAY_SDI: now also J4.8
- net GND: now also IC2.F4 (VSS_7), IC2.F5 (VSS_8), R14.2, R8.2, U11.1 (STAT), C17.2, C20.2, C21.2, C22.2, C23.2, IC4.1 (GND_1), IC4.4 (~{ON}), IC4.5 (GND_2), J4.15, J4.5, U12.3 (GND), U12.7 (PAD), U3.12 (GND), U3.4 (PGND); no longer R8.1
- net GPS_EXTINT: now also IC2.C4 (P1.01); no longer IC2.A2 (P0.12/TRACECLK/DCX), IC2.B5 (P0.03/NFC2)
- net GPS_RX: now also IC2.A4 (P1.00); no longer IC2.A5 (P0.20)
- net GPS_TX: now also IC2.A5 (P0.20); no longer IC2.A4 (P1.00)
- net HR_INT: now also U3.13 (~{INT})
- net INT1_BMI270: now also IC2.G3 (P0.25/AIN4); no longer IC2.J4 (N/C_3)
- net INT2_BMI270: now also IC2.G4 (P1.04); no longer IC2.J5 (N/C_4)
- net LEDK: now also J4.14
- net LIS2MDLTR_INT: now also IC2.H3 (P0.27/AIN6); no longer IC2.J3 (RESET_N)
- net RTC Battery: now also U10.6 (VBACKUP), C17.1, C20.1
- net RTC_INT: no longer U10.2 (~{INT})
- net SCL: now also R15.1; no longer R14.1
- net SDA: now also R10.1; no longer R13.1
- net TP_INT: now also IC2.E9 (P1.05), J4.3; no longer IC2.D8 (P0.04/AIN0)
- net TP_RST: now also J4.4
- net VIN_SWD: now also IC4.6 (VIN2); no longer IC2.B9 (VBUS), IC3.3 (VIN1), J1.1 (Pin_1), U11.4 (V_{DD})
- net at R7.2, U5.7 (EXTINT0): now also R8.1; no longer R8.2
- net at U5.16 (RF_OUT): now also R2.2; no longer R2.1
- net at U5.17 (RF_IN): now also R2.1; no longer R2.2
- net at U5.28 (FORCE_ON): now also R13.2, R14.1
- net TWI_SCL: now reaches IC2.A3 (P1.03/TWI)
- net TWI_SCL: now also J4.1, R16.2, U3.2 (SCL)
- net TWI_SDA: now reaches IC2.B4 (P1.02/TWI)
- net TWI_SDA: now also J4.2, R12.2, U3.3 (SDA)
- net GPS_FORCEON: now reaches IC2.C5 (P0.02/NFC1)
- net GPS_FORCEON: now also R13.1
- net HR_LED_EN: now reaches IC2.F3 (P0.19)
- net HR_LED_EN: now also U12.4 (EN)
- net VBUS renamed VDD
- net VDD: now also C16.1, C22.1, U12.6 (IN)
- new net +5V: C21.1, C4.1, C5.1, U12.1 (OUT), U3.10 (VLED+), U3.9 (VLED+)
- new net VIN: IC3.3 (VIN1), IC4.2 (VOUT_1), IC4.7 (VOUT_2), U11.4 (V_{DD})
- new net VIN_USB: IC2.B9 (VBUS), IC4.3 (VIN1), J1.1 (Pin_1)
- no-connect marks 44 -> 42
Other:
- note added: "Accelerometer"
- note added: "Battery Charger & Gauge"
- note added: "HR & Oximeter Sensor"
- note added: "I2C Pullups"
- note added: "Power Path"
- note removed: "Accelerometer & Gyroscope"
- note removed: "Battery Gauge"
- note removed: "Charging Circuit"
- note removed: "Heart-Rate Sensor"
- moved on the sheet: BT1, BT2, C1, C10, C11, C12, C13, C14, C15, C18, C19, C2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

Commit message: -
Parts:
- added E1: W3010, W3010:XCVR_W3010, symbol W3010:W3010
- added U13: MIA-M10Q-00B, MIA-M10Q-00B:LGA_M10Q-00B_UBL, symbol MIA-M10Q-00B:MIA-M10Q-00B
- C11, C12, C13, C14, C18, C3: footprint Capacitor_SMD:C_0402_1005Metric -> Capacitor_SMD:C_0201_0603Metric
- R10, R12, R15, R16: footprint Resistor_SMD:R_0402_1005Metric -> Resistor_SMD:R_0201_0603Metric
Changed lines of the file:
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@@
       (effects (font (size 1.27 1.27)) (justify left))
     )
-    (property "Footprint" "Capacitor_SMD:C_0402_1005Metric" (at 341.0573 354.7078 0)
+    (property "Footprint" "Capacitor_SMD:C_0201_0603Metric" (at 341.0573 354.7078 0)
       (effects (font (size 1.27 1.27)) hide)
     )
@@
       (effects (font (size 1.27 1.27)) (justify left))
     )
-    (property "Footprint" "Capacitor_SMD:C_0402_1005Metric" (at 153.3764 281.0093 0)
+    (property "Footprint" "Capacitor_SMD:C_0201_0603Metric" (at 153.3764 281.0093 0)
       (effects (font (size 1.27 1.27)) hide)
     )
@@
       (effects (font (size 1.27 1.27)))
     )
-    (property "Footprint" "Resistor_SMD:R_0402_1005Metric" (at 513.08 348.742 90)
+    (property "Footprint" "Resistor_SMD:R_0201_0603Metric" (at 513.08 348.742 90)
       (effects (font (size 1.27 1.27)) hide)
     )
@@
     )
   )
+  (symbol (lib_id "MIA-M10Q-00B:MIA-M10Q-00B") (at 184.507 219.6744 0) (unit 1)
+    (in_bom yes) (on_board yes) (dnp no) (fields_autoplaced)
+    (property "Reference" "U13" (at 214.987 209.55 0)
+      (effects (font (size 1.524 1.524)))
+    )
+    (property "Value" "MIA-M10Q-00B" (at 214.987 212.09 0)
+      (effects (font (size 1.524 1.524)))
+    )
+    (property "Footprint" "MIA-M10Q-00B:LGA_M10Q-00B_UBL" (at 184.507 219.6744 0)
+      (effects (font (size 1.27 1.27) italic) hide)
+    )
+    (property "Datasheet" "MIA-M10Q-00B" (at 184.507 219.6744 0)
+      (effects (font (size 1.27 1.27) italic) hide)
+    )
+    (pin "A1")
+    (pin "A2")
+    (pin "A3")
+    (pin "A4")
+    (pin "A5")
+    (pin "A6")
+    (pin "A7")
+    (pin "A8")
+    (pin "A9")
+    (pin "B1")
+    (pin "B2")
+    (pin "B8")
+    (pin "B9")
+    (pin "C1")
+    (pin "C3")
+    (pin "C4")
+    (pin "C5")
+    (pin "C6")
+    (pin "C7")
+    (pin "C9")
+    (pin "D1")
+    (pin "D2")
+    (pin "D9")
+    (pin "E1")
+    (pin "E2")
+    (pin "E3")
+    (pin "E4")
+    (pin "E7")
+    (pin "E9")
+    (pin "F1")
+    (pin "F3")
+    (pin "F4")
+    (pin "F7")
+    (pin "F9")
+    (pin "G1")
+    (pin "G3")
+    (pin "G4")
+    (pin "G5")
+    (pin "G6")
+    (pin "G7")
+    (pin "G9")
+    (pin "H1")
+    (pin "H8")
+    (pin "H9")
+    (pin "J1")
+    (pin "J2")
+    (pin "J3")
+    (pin "J4")
+    (pin "J5")
+    (pin "J6")
+    (pin "J7")
+    (pin "J8")
+    (pin "J9")
+    (instances
+      (project "smartwatch"
+        (path "/66aaca1a-81b1-4743-8182-fb4c70cf8a2a"
+          (reference "U13") (unit 1)
+        )
+      )
+    )
+  )
   (symbol (lib_id "Device:C") (at 58.8682 91.8302 0) (unit 1)
     (in_bom yes) (on_board yes) (dnp no)
@@
       (effects (font (size 1.27 1.27)) (justify left))
     )
-    (property "Footprint" "Capacitor_SMD:C_0402_1005Metric" (at 453.8872 357.8145 0)
+    (property "Footprint" "Capacitor_SMD:C_0201_0603Metric" (at 453.8872 357.8145 0)
       (effects (font (size 1.27 1.27)) hide)
     )
@@
       (effects (font (size 1.27 1.27)) (justify left))
     )
-    (property "Footprint" "Capacitor_SMD:C_0402_1005Metric" (at 444.3983 357.7228 0)
+    (property "Footprint" "Capacitor_SMD:C_0201_0603Metric" (at 444.3983 357.7228 0)
       (effects (font (size 1.27 1.27)) hide)
     )
@@
       (effects (font (size 1.27 1.27)))
     )
-    (property "Footprint" "Resistor_SMD:R_0402_1005Metric" (at 513.1442 340.47 90)
+    (property "Footprint" "Resistor_SMD:R_0201_0603Metric" (at 513.1442 340.47 90)
       (effects (font (size 1.27 1.27)) hide)
     )
@@
       (effects (font (size 1.27 1.27)) (justify left))
     )
-    (property "Footprint" "Capacitor_SMD:C_0402_1005Metric" (at 433.7753 364.9287 0)
+    (property "Footprint" "Capacitor_SMD:C_0201_0603Metric" (at 433.7753 364.9287 0)
       (effects (font (size 1.27 1.27)) hide)
     )
@@
       (effects (font (size 1.27 1.27)))
     )
-    (property "Footprint" "Resistor_SMD:R_0402_1005Metric" (at 540.8637 340.2812 90)
+    (property "Footprint" "Resistor_SMD:R_0201_0603Metric" (at 540.8637 340.2812 90)
       (effects (font (size 1.27 1.27)) hide)
     )
@@
       (effects (font (size 1.27 1.27)) (justify left))
     )
-    (property "Footprint" "Capacitor_SMD:C_0402_1005Metric" (at 334.6828 354.729 0)
+    (property "Footprint" "Capacitor_SMD:C_0201_0603Metric" (at 334.6828 354.729 0)
       (effects (font (size 1.27 1.27)) hide)
     )
@@
       (effects (font (size 1.27 1.27)))
     )
-    (property "Footprint" "Resistor_SMD:R_0402_1005Metric" (at 540.7817 348.8062 90)
+    (property "Footprint" "Resistor_SMD:R_0201_0603Metric" (at 540.7817 348.8062 90)
       (effects (font (size 1.27 1.27)) hide)
     )
@@
         )
       )
+    )
+  )
+  (symbol (lib_id "W3010:W3010") (at 245.8731 224.1158 0) (unit 1)
+    (in_bom yes) (on_board yes) (dnp no) (fields_autoplaced)
+    (property "Reference" "E1" (at 248.92 223.2903 0)
+      (effects (font (size 1.27 1.27)) (justify left))
+    )
+    (property "Value" "W3010" (at 248.92 225.8303 0)
+      (effects (font (size 1.27 1.27)) (justify left))
+    )
+    (property "Footprint" "W3010:XCVR_W3010" (at 245.8731 224.1158 0)
+      (effects (font (size 1.27 1.27)) (justify bottom) hide)
+    )
+    (property "Datasheet" "" (at 245.8731 224.1158 0)
+      (effects (font (size 1.27 1.27)) hide)
+    )
+    (property "PARTREV" "L192.C 2/16" (at 245.8731 224.1158 0)
+      (effects (font (size 1.27 1.27)) (justify bottom) hide)
+    )
+    (property "MANUFACTURER" "Pulse" (at 245.8731 224.1158 0)
+      (effects (font (size 1.27 1.27)) (justify bottom) hide)
+    )
+    (property "MAXIMUM_PACKAGE_HEIGHT" "2mm" (at 245.8731 224.1158 0)
+      (effects (font (size 1.27 1.27)) (justify bottom) hide)
+    )
+    (property "STANDARD" "Manufacturer Recommendations" (at 245.8731 224.1158 0)
+      (effects (font (size 1.27 1.27)) (justify bottom) hide)
+    )
+    (pin "1")
+    (pin "2")
+    (instances
+      (project "smartwatch"
+        (path "/66aaca1a-81b1-4743-8182-fb4c70cf8a2a"
+          (reference "E1") (unit 1)
+        )
+      )
